File: ember-pcb.kicad_sch (KiCad schematic)
At the start: 36 parts, among them J1 Samtec_ASP-134602-01, J2 Conn_Coaxial_Power, J3 Conn_02x12_Odd_Even, J4 Conn_01x07, J5 Conn_Coaxial_Power, SW1 SW_SP3T, SW2 SW_SP3T, SW3 SW_DIP_x02, U1 EMBER Macro, U2 LP5912-0.9DRV, U3 LP5912-1.1DRV, U4 LP5912-2.5DRV

Commit message: Updates
Parts:
- added J2: Conn_02x06_Odd_Even, Connector_PinHeader_2.54mm:PinHeader_2x06_P2.54mm_Vertical, symbol Connector_Generic:Conn_02x06_Odd_Even
- renumbered J2 to J3, J3 to J4, J4 to J5, J5 to J6, SW3 to SW2, SW2 to SW3
Connections:
- net GND: now also J2.10 (Pin_10), J2.9 (Pin_9); no longer U1.A19 (vss), U1.B8 (vss)
- net bl_source_pin: now also U1.B8 (bl_source_pin)
- net io_pwr: no longer SW2.3, SW2.4
- net mclk_pause: now also J2.6 (Pin_6); no longer J1.K29 (Pin_29)
- net miso: now also J2.7 (Pin_7); no longer J1.E36 (Pin_36)
- net mosi: now also J2.5 (Pin_5); no longer J1.E30 (Pin_30)
- net rst_n: now also J2.2 (Pin_2); no longer J1.D26 (Pin_26)
- net sc: now also J2.1 (Pin_1); no longer J1.E34 (Pin_34)
- net sclk: now also J2.3 (Pin_3); no longer J1.K28 (Pin_28)
- net sl_source_pin: now also U1.B3 (sl_source_pin)
- net vddio_fsm: no longer U1.B3 (vddio_fsm)
- net vadj: now reaches J5.6 (Pin_6)
- net vadj: now also J1.E39 (Pin_39), J1.F40 (Pin_40), J1.G39 (Pin_39), J1.H40 (Pin_40), J1.J39 (Pin_39), J1.K40 (Pin_40), SW2.3, SW2.4
- new net rram_busy: J2.4 (Pin_4), U1.A19 (rram_busy)
- no-connect marks 81 -> 83
Other:
- note added: "GND CLK1_M2C_P CLK1_M2C_N GND GND LA00_P_CC LA00_N_CC GND LA03_P LA03_N GND LA08_P LA08_N GND LA12_P LA12_N GND LA16_P LA16_N GND LA20_P LA20_N GND LA22_P LA22_N GND LA25_P LA25_N GND LA29_P LA29_N GND LA31_P LA31_N GND LA33_P LA33_N GND vadj GND"
- note added: "GND HA01_P_CC HA01_N_CC GND GND HA05_P HA05_N GND HA09_P HA09_N GND HA13_P HA13_N GND HA16_P HA16_N GND HA20_P HA20_N GND HB03_P HB03_N GND HB05_P HB05_N GND HB09_P HB09_N GND HB13_P HB13_N GND HB19_P HB19_N GND HB21_P HB21_N GND vadj GND"
- note added: "PG_M2C GND GND HA00_P_CC HA00_N_CC GND HA04_P HA04_N GND HA08_P HA08_N GND HA12_P HA12_N GND HA15_P HA15_N GND HA19_P HA19_N GND HB02_P HB02_N GND HB04_P HB04_N GND HB08_P HB08_N GND HB12_P HB12_N GND HB16_P HB16_N GND HB20_P HB20_N GND vadj"
- note added: "PMOD Header"
- note added: "VREF_A_M2C PRSNT_M2C_L GND CLK0_M2C_P CLK0_M2C_N GND LA02_P LA02_N GND LA04_P LA04_N GND LA07_P LA07_N GND LA11_P LA11_N GND LA15_P LA15_N GND LA19_P LA19_N GND LA21_P LA21_N GND LA24_P LA24_N GND LA28_P LA28_N GND LA30_P LA30_N GND LA32_P LA32_N GND vadj"
- note removed: "GND CLK1_M2C_P CLK1_M2C_N GND GND LA00_P_CC LA00_N_CC GND LA03_P LA03_N GND LA08_P LA08_N GND LA12_P LA12_N GND LA16_P LA16_N GND LA20_P LA20_N GND LA22_P LA22_N GND LA25_P LA25_N GND LA29_P LA29_N GND LA31_P LA31_N GND LA33_P LA33_N GND VADJ GND"
- note removed: "GND HA01_P_CC HA01_N_CC GND GND HA05_P HA05_N GND HA09_P HA09_N GND HA13_P HA13_N GND HA16_P HA16_N GND HA20_P HA20_N GND HB03_P HB03_N GND HB05_P HB05_N GND HB09_P HB09_N GND HB13_P HB13_N GND HB19_P HB19_N GND HB21_P HB21_N GND VADJ GND"
- note removed: "PG_M2C GND GND HA00_P_CC HA00_N_CC GND HA04_P HA04_N GND HA08_P HA08_N GND HA12_P HA12_N GND HA15_P HA15_N GND HA19_P HA19_N GND HB02_P HB02_N GND HB04_P HB04_N GND HB08_P HB08_N GND HB12_P HB12_N GND HB16_P HB16_N GND HB20_P HB20_N GND VADJ"
- note removed: "VREF_A_M2C PRSNT_M2C_L GND CLK0_M2C_P CLK0_M2C_N GND LA02_P LA02_N GND LA04_P LA04_N GND LA07_P LA07_N GND LA11_P LA11_N GND LA15_P LA15_N GND LA19_P LA19_N GND LA21_P LA21_N GND LA24_P LA24_N GND LA28_P LA28_N GND LA30_P LA30_N GND LA32_P LA32_N GND VADJ"
- moved on the sheet: FID1, FID2, FID3, H1, H2, H3, H4, J4, J5, R2, R3, SW2

Commit message: Fixes
Connections:
- net GND: now also J3.2 (Ext), J6.2 (Ext); no longer J3.1 (In), J6.1 (In)
- net at SW3.1: now also J6.1 (In); no longer J6.2 (Ext)
- net at SW1.1: now also J3.1 (In); no longer J3.2 (Ext)
Other:
- moved on the sheet: J3, J6
Changed lines of the file:
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@@
     (pin "1")
   )
-  (symbol (lib_id "Connector:Conn_Coaxial_Power") (at 59.69 332.74 90) (unit 1)
+  (symbol (lib_id "Connector:Conn_Coaxial_Power") (at 62.23 332.74 270) (unit 1)
     (in_bom yes) (on_board yes) (fields_autoplaced)
-    (property "Reference" "J3" (id 0) (at 61.214 326.39 90))
-    (property "Value" "Conn_Coaxial_Power" (id 1) (at 61.214 328.93 90))
+    (property "Reference" "J3" (id 0) (at 60.706 326.39 90))
+    (property "Value" "Conn_Coaxial_Power" (id 1) (at 60.706 328.93 90))
     (property "Footprint" "Connector_Coaxial:SMA_Molex_73251-2200_Horizontal" (id 2) (at 60.96 332.74 0)
       (effects (font (size 1.27 1.27)) hide)
@@
     (pin "1")
   )
-  (symbol (lib_id "Connector:Conn_Coaxial_Power") (at 65.405 370.205 90) (unit 1)
+  (symbol (lib_id "Connector:Conn_Coaxial_Power") (at 67.945 370.205 270) (unit 1)
     (in_bom yes) (on_board yes) (fields_autoplaced)
-    (property "Reference" "J6" (id 0) (at 66.929 363.855 90))
-    (property "Value" "Conn_Coaxial_Power" (id 1) (at 66.929 366.395 90))
+    (property "Reference" "J6" (id 0) (at 66.421 363.22 90))
+    (property "Value" "Conn_Coaxial_Power" (id 1) (at 66.421 365.76 90))
     (property "Footprint" "Connector_Coaxial:SMA_Molex_73251-2200_Horizontal" (id 2) (at 66.675 370.205 0)
       (effects (font (size 1.27 1.27)) hide)

Commit message: Updates
Parts:
- removed SW2: SW_DIP_x02, Button_Switch_SMD:SW_DIP_SPSTx02_Slide_Omron_A6S-210x_W8.9mm_P2.54mm, symbol Switch:SW_DIP_x02
- removed U2: LP5912-0.9DRV, Package_SON:WSON-6-1EP_2x2mm_P0.65mm_EP1x1.6mm_ThermalVias, symbol Regulator_Linear:LP5912-0.9DRV
- removed U3: LP5912-1.1DRV, Package_SON:WSON-6-1EP_2x2mm_P0.65mm_EP1x1.6mm_ThermalVias, symbol Regulator_Linear:LP5912-1.1DRV
- removed U4: LP5912-2.5DRV, Package_SON:WSON-6-1EP_2x2mm_P0.65mm_EP1x1.6mm_ThermalVias, symbol Regulator_Linear:LP5912-2.5DRV
- added C11, C12: 27pF, Capacitor_SMD:C_0603_1608Metric, symbol Device:C
- added C13: 4.7u, Capacitor_Tantalum_SMD:CP_EIA-3528-12_Kemet-T, symbol Device:C_Polarized
- added C14: 100nF, Capacitor_SMD:C_1210_3225Metric, symbol Device:C
- added D2: LED, LED_SMD:LED_0603_1608Metric, symbol Device:LED
- added H5, H6: MountingHole, MountingHole:MountingHole_3mm_Pad, symbol Mechanical:MountingHole_Pad
- added J7: USB_B_Micro, Connector_USB:USB_Micro-B_Molex-105017-0001, symbol Connector:USB_B_Micro
- added J8, J9: Conn_Coaxial_Power, Connector_Coaxial:SMA_Molex_73251-2200_Horizontal, symbol Connector:Conn_Coaxial_Power
- added R4: 10k, Resistor_SMD:R_0603_1608Metric, symbol Device:R
- added R5: 1k, Resistor_SMD:R_0603_1608Metric, symbol Device:R
- added R6: 1M, Resistor_SMD:R_0603_1608Metric, symbol Device:R
- added R7: 12k, Resistor_SMD:R_0603_1608Metric, symbol Device:R
- added R8: 47k, Resistor_SMD:R_0603_1608Metric, symbol Device:R
- added SW2: SW_DIP_x03, Button_Switch_SMD:SW_DIP_SPSTx03_Slide_Omron_A6S-310x_W8.9mm_P2.54mm, symbol Switch:SW_DIP_x03
- added U2: TLV71209_SOT23-5, Package_TO_SOT_SMD:SOT-23-5, symbol Regulator_Linear:TLV71209_SOT23-5
- added U3: TLV71211_SOT23-5, Package_TO_SOT_SMD:SOT-23-5, symbol Regulator_Linear:TLV71211_SOT23-5
- added U4: FT4222HQ, Package_DFN_QFN:VQFN-32-1EP_5x5mm_P0.5mm_EP3.1x3.1mm, symbol Interface_USB:FT4222HQ
- added Y1: 12MHz, Crystal:Crystal_SMD_0603-2Pin_6.0x3.5mm, symbol Device:Crystal
Connections:
- net +3.3V: now also R4.1, R8.1, U2.1 (IN), U2.3 (EN), U3.1 (IN), U3.3 (EN), U4.25 (VOUT3V3), U4.7 (VCCIO)
- net GND: now also C11.2, C12.2, C13.2, C14.2, D2.1 (K), H5.1, H6.1, J7.4 (ID), J7.5 (GND), J7.6 (Shield), R7.1, U2.2 (GND), U3.2 (GND), U4.20 (UGND), U4.24 (UGND), U4.27 (AGND), U4.28 (DGND), U4.33 (EP), U4.4 (DCNF0), U4.5 (DCNF1), U4.6 (DGND)
- net aclk: no longer J1.K25 (Pin_25)
- net bl_en: no longer J1.E27 (Pin_27)
- net bleed_en: no longer J1.J19 (Pin_19)
- net bsl_dac_config_0: no longer J1.H29 (Pin_29)
- net bsl_dac_config_1: no longer J1.E33 (Pin_33)
- net bsl_dac_config_2: no longer J1.F29 (Pin_29)
- net bsl_dac_config_3: no longer J1.K32 (Pin_32)
- net bsl_dac_config_4: no longer J1.J33 (Pin_33)
- net bsl_dac_en: no longer J1.J28 (Pin_28)
- net byp: now also SW2.2
- net clamp_ref_0: no longer J1.K35 (Pin_35)
- net clamp_ref_1: no longer J1.J27 (Pin_27)
- net clamp_ref_2: no longer J1.H28 (Pin_28)
- net clamp_ref_3: no longer J1.F26 (Pin_26)
- net clamp_ref_4: no longer J1.G27 (Pin_27)
- net clamp_ref_5: no longer J1.G25 (Pin_25)
- net di_0: no longer J1.F25 (Pin_25)
- net di_1: no longer J1.D27 (Pin_27)
- net di_10: no longer J1.F22 (Pin_22)
- net di_11: no longer J1.C22 (Pin_22)
- net di_12: no longer J1.H20 (Pin_20)
- net di_13: no longer J1.D21 (Pin_21)
- net di_14: no longer J1.E19 (Pin_19)
- net di_15: no longer J1.K20 (Pin_20)
- net di_16: no longer J1.C18 (Pin_18)
- net di_17: no longer J1.F19 (Pin_19)
- net di_18: no longer J1.K16 (Pin_16)
- net di_19: no longer J1.H19 (Pin_19)
- net di_2: no longer J1.G24 (Pin_24)
- net di_20: no longer J1.G19 (Pin_19)
- net di_21: no longer J1.D18 (Pin_18)
- net di_22: no longer J1.E18 (Pin_18)
- net di_23: no longer J1.F14 (Pin_14)
- net di_24: no longer J1.D17 (Pin_17)
- net di_25: no longer J1.J15 (Pin_15)
- net di_26: no longer J1.F17 (Pin_17)
- net di_27: no longer J1.C11 (Pin_11)
- net di_28: no longer J1.E16 (Pin_16)
- net di_29: no longer J1.F16 (Pin_16)
- net di_3: no longer J1.C26 (Pin_26)
- net di_30: no longer J1.H14 (Pin_14)
- net di_31: no longer J1.K14 (Pin_14)
- net di_32: no longer J1.D11 (Pin_11)
- net di_33: no longer J1.F11 (Pin_11)
- net di_34: no longer J1.J6 (Pin_6)
- net di_35: no longer J1.H11 (Pin_11)
- net di_36: no longer J1.E2 (Pin_2)
- net di_37: no longer J1.F8 (Pin_8)
- net di_38: no longer J1.K11 (Pin_11)
- net di_39: no longer J1.H8 (Pin_8)
- net di_4: no longer J1.E24 (Pin_24)
- net di_40: no longer J1.D12 (Pin_12)
- net di_41: no longer J1.K8 (Pin_8)
- net di_42: no longer J1.D9 (Pin_9)
- net di_43: no longer J1.E12 (Pin_12)
- net di_44: no longer J1.E9 (Pin_9)
- net di_45: no longer J1.G9 (Pin_9)
- net di_46: no longer J1.G12 (Pin_12)
- net di_47: no longer J1.E3 (Pin_3)
- net di_5: no longer J1.C23 (Pin_23)
- net di_6: no longer J1.D23 (Pin_23)
- net di_7: no longer J1.K22 (Pin_22)
- net di_8: no longer J1.D24 (Pin_24)
- net di_9: no longer J1.E22 (Pin_22)
- net man: now also SW2.1
- net mclk_pause: now also J1.H34 (Pin_34), U4.13 (GPIO0)
- net miso: now also J1.H37 (Pin_37), J2.5 (Pin_5), U4.9 (MISO); no longer J2.7 (Pin_7)
- net mosi: now also J1.G37 (Pin_37), J2.3 (Pin_3), U4.10 (MOSI); no longer J2.5 (Pin_5)
- net read_dac_config_0: no longer J1.D8 (Pin_8)
- net read_dac_config_1: no longer J1.C15 (Pin_15)
- net read_dac_config_2: no longer J1.D14 (Pin_14)
- net read_dac_config_3: no longer J1.G16 (Pin_16)
- net read_dac_en: no longer J1.H32 (Pin_32)
- net read_ref_0: no longer J1.J12 (Pin_12)
- net read_ref_1: no longer J1.F7 (Pin_7)
- net read_ref_2: no longer J1.G7 (Pin_7)
- net read_ref_3: no longer J1.E13 (Pin_13)
- net read_ref_4: no longer J1.F4 (Pin_4)
- net read_ref_5: no longer J1.C10 (Pin_10)
- net rram_addr_0: no longer J1.F5 (Pin_5)
- net rram_addr_1: no longer J1.H7 (Pin_7)
- net rram_addr_10: no longer J1.G6 (Pin_6)
- net rram_addr_11: no longer J1.H10 (Pin_10)
- net rram_addr_12: no longer J1.J13 (Pin_13)
- net rram_addr_13: no longer J1.J10 (Pin_10)
- net rram_addr_14: no longer J1.K13 (Pin_13)
- net rram_addr_15: no longer J1.K10 (Pin_10)
- net rram_addr_2: no longer J1.E6 (Pin_6)
- net rram_addr_3: no longer J1.F13 (Pin_13)
- net rram_addr_4: no longer J1.E10 (Pin_10)
- net rram_addr_5: no longer J1.F10 (Pin_10)
- net rram_addr_6: no longer J1.J7 (Pin_7)
- net rram_addr_7: no longer J1.G13 (Pin_13)
- net rram_addr_8: no longer J1.G10 (Pin_10)
- net rram_addr_9: no longer J1.H13 (Pin_13)
- net rram_busy: now also J1.H35 (Pin_35), J2.2 (Pin_2), U4.14 (GPIO1); no longer J2.4 (Pin_4)
- net rst_n: now also J1.H38 (Pin_38), J2.4 (Pin_4); no longer J2.2 (Pin_2)
- net sa_clk: now also J1.K4 (Pin_4); no longer J1.K37 (Pin_37)
- net sa_do_0: no longer J1.D20 (Pin_20)
- net sa_do_1: no longer J1.G21 (Pin_21)
- net sa_do_10: no longer J1.G33 (Pin_33)
- net sa_do_11: no longer J1.F23 (Pin_23)
- net sa_do_12: no longer J1.H23 (Pin_23)
- net sa_do_13: no longer J1.E25 (Pin_25)
- net sa_do_14: no longer J1.J24 (Pin_24)
- net sa_do_15: no longer J1.G28 (Pin_28)
- net sa_do_16: no longer J1.J25 (Pin_25)
- net sa_do_17: no longer J1.C27 (Pin_27)
- net sa_do_18: no longer J1.H25 (Pin_25)
- net sa_do_19: no longer J1.F32 (Pin_32)
- net sa_do_2: no longer J1.C19 (Pin_19)
- net sa_do_20: no longer J1.K26 (Pin_26)
- net sa_do_21: no longer J1.H26 (Pin_26)
- net sa_do_22: no longer J1.F28 (Pin_28)
- net sa_do_23: no longer J1.E28 (Pin_28)
- net sa_do_24: no longer J1.K31 (Pin_31)
- net sa_do_25: no longer J1.J31 (Pin_31)
- net sa_do_26: now also J1.H28 (Pin_28); no longer J1.H37 (Pin_37)
- net sa_do_27: no longer J1.H31 (Pin_31)
- net sa_do_28: no longer J1.H35 (Pin_35)
- net sa_do_29: no longer J1.G31 (Pin_31)
- net sa_do_3: no longer J1.E21 (Pin_21)
- net sa_do_30: no longer J1.F35 (Pin_35)
- net sa_do_31: no longer J1.G37 (Pin_37)
- net sa_do_32: no longer J1.F31 (Pin_31)
- net sa_do_33: no longer J1.K34 (Pin_34)
- net sa_do_34: no longer J1.J34 (Pin_34)
- net sa_do_35: now also J1.H31 (Pin_31); no longer J1.K38 (Pin_38)
- net sa_do_36: no longer J1.E31 (Pin_31)
- net sa_do_37: no longer J1.H34 (Pin_34)
- net sa_do_38: no longer J1.G34 (Pin_34)
- net sa_do_39: no longer J1.J30 (Pin_30)
- net sa_do_4: no longer J1.F20 (Pin_20)
- net sa_do_40: now also J1.H32 (Pin_32); no longer J1.H38 (Pin_38)
- net sa_do_41: now also J1.H29 (Pin_29); no longer J1.E37 (Pin_37)
- net sa_do_42: no longer J1.F37 (Pin_37)
- net sa_do_43: no longer J1.F34 (Pin_34)
- net sa_do_44: now also J1.G33 (Pin_33); no longer J1.F38 (Pin_38)
- net sa_do_45: no longer J1.G30 (Pin_30)
- net sa_do_46: now also J1.G34 (Pin_34); no longer J1.J37 (Pin_37)
- net sa_do_47: now also J1.G30 (Pin_30); no longer J1.J36 (Pin_36)
- net sa_do_5: no longer J1.J21 (Pin_21)
- net sa_do_6: no longer J1.J22 (Pin_22)
- net sa_do_7: no longer J1.G22 (Pin_22)
- net sa_do_8: no longer J1.H22 (Pin_22)
- net sa_do_9: no longer J1.K23 (Pin_23)
- net sa_en: no longer J1.E7 (Pin_7)
- net sa_rdy: now also J1.G31 (Pin_31); no longer J1.G36 (Pin_36)
- net sc: now also J1.G36 (Pin_36), U4.32 (~{SS})
- net sclk: now also J1.C22 (Pin_22), J2.7 (Pin_7), U4.8 (SCK); no longer J2.3 (Pin_3)
- net set_rst: no longer J1.J9 (Pin_9)
- net sl_en: no longer J1.K7 (Pin_7)
- net vadj: now also J1.H1 (Pin_1), J1.K1 (Pin_1), SW3.4, SW2.5, SW2.6
- net vddio: now also SW2.4
- net we: no longer J1.C14 (Pin_14)
- net wl_dac_config_0: no longer J1.D15 (Pin_15)
- net wl_dac_config_1: no longer J1.H17 (Pin_17)
- net wl_dac_config_2: no longer J1.H16 (Pin_16)
- net wl_dac_config_3: no longer J1.E15 (Pin_15)
- net wl_dac_config_4: no longer J1.K17 (Pin_17)
- net wl_dac_config_5: no longer J1.G15 (Pin_15)
- net wl_dac_config_6: no longer J1.G18 (Pin_18)
- net wl_dac_config_7: no longer J1.J16 (Pin_16)
- net wl_dac_en: no longer J1.J18 (Pin_18)
- net wl_en: no longer J1.K19 (Pin_19)
- net wl_source_pin: now also SW2.3
- net at SW1.2: now also U3.5 (OUT)
- net at J1.F1 (Pin_1): now also R5.2
- net dp0_c2m_p: now reaches J1.C2 (Pin_2)
- net dp0_c2m_n: now reaches J1.C3 (Pin_3)
- net dp0_m2c_p: now reaches J1.C6 (Pin_6)
- net dp0_m2c_n: now reaches J1.C7 (Pin_7)
- net clk0_m2c_p: now reaches J1.H4 (Pin_4)
- net clk0_m2c_p: now also J8.1 (In)
- net clk0_m2c_n: now reaches J1.H5 (Pin_5)
- net clk0_m2c_n: now also J8.2 (Ext)
- net at J1.B1 (Pin_1): now also R4.2
- net at SW1.4: now also U2.5 (OUT)
- net clk1_m2c_p: now reaches J1.G2 (Pin_2)
- net clk1_m2c_p: now also J9.1 (In)
- net clk1_m2c_n: now reaches J1.G3 (Pin_3)
- net clk1_m2c_n: now also J9.2 (Ext)
- new net: C13.1, C14.1, J7.1 (VBUS), U4.26 (VCCIN), U4.30 (VBUS_DET)
- new net: J7.2 (D-), U4.22 (DM)
- new net: J7.3 (D+), U4.23 (DP)
- new net: R8.2, U4.1 (DEBUGGER), U4.2 (~{STEST_RST}), U4.3 (~{RESET})
- new net: C11.1, R6.1, U4.18 (XSCI), Y1.1
- new net: C12.1, R6.2, U4.19 (XSCO), Y1.2
- new net: R7.2, U4.21 (RREF)
- new net: D2.2 (A), R5.1
- no-connect marks 83 -> 68
Other:
- note added: "USB SPI"
- note removed: "PMOD Header"
- moved on the sheet: C1, C10, C2, C3, C4, C5, C6, C7, C8, C9, FB1, FB2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
